File: pcb/prototype1/prototype1.sch (KiCad schematic (older format))
At the start: 66 parts, among them P1 USB_B, P2 AAA1 HOT, P3 AAA1 GND, P4 AAA2 GND, P5 AAA2 HOT, SW1 UP/BOOT, SW2 LEFT, SW3 RIGHT, SW4 DOWN, SW5 SPST, U1 STM32F410R8-LQFP64, U2 TLC5926, U3 TLC5926, U4 TLC5926, U5 LM1117-3.3, U6 TPS61021

Commit message: fix custom kicad libs
Parts:
- LED1, LED10, LED11, LED12, LED13, LED14, LED15, LED16, LED17, LED18, LED19, LED2, LED20, LED21, LED22, LED23, LED24, LED25, LED26, LED27, LED28, LED29, LED3, LED30, LED31, LED32, LED4, LED5, LED6, LED7, LED8, LED9: footprint spinny:LED_CLV1L-PLCC4 -> spin:LED_CLV1L-PLCC4
Changed lines of the file:
@@
 EESchema Schematic File Version 2
-LIBS:prototype1-rescue
+LIBS:spin
 LIBS:power
 LIBS:device
@@
 LIBS:contrib
 LIBS:valves
-LIBS:stm32f410r8-lqfp64
-LIBS:prototype1-cache
 EELAYER 25 0
 EELAYER END
@@
 F 0 "LED1" H 9150 600 60  0000 C CNN
 F 1 "RGB" H 9600 600 60  0000 C CNN
-F 2 "spinny:LED_CLV1L-PLCC4" H 9400 400 60  0001 C CNN
+F 2 "spin:LED_CLV1L-PLCC4" H 9400 400 60  0001 C CNN
 F 3 "" H 9400 400 60  0000 C CNN
 	1    9400 600
@@
 F 0 "LED2" H 9150 850 60  0000 C CNN
 F 1 "RGB" H 9600 850 60  0000 C CNN
-F 2 "spinny:LED_CLV1L-PLCC4" H 9400 650 60  0001 C CNN
+F 2 "spin:LED_CLV1L-PLCC4" H 9400 650 60  0001 C CNN
 F 3 "" H 9400 650 60  0000 C CNN
 	1    9400 850
@@
 F 0 "LED3" H 9150 1100 60  0000 C CNN
 F 1 "RGB" H 9600 1100 60  0000 C CNN
-F 2 "spinny:LED_CLV1L-PLCC4" H 9400 900 60  0001 C CNN
+F 2 "spin:LED_CLV1L-PLCC4" H 9400 900 60  0001 C CNN
 F 3 "" H 9400 900 60  0000 C CNN
 	1    9400 1100
@@
 F 0 "LED4" H 9150 1350 60  0000 C CNN
 F 1 "RGB" H 9600 1350 60  0000 C CNN
-F 2 "spinny:LED_CLV1L-PLCC4" H 9400 1150 60  0001 C CNN
+F 2 "spin:LED_CLV1L-PLCC4" H 9400 1150 60  0001 C CNN
 F 3 "" H 9400 1150 60  0000 C CNN
 	1    9400 1350
@@
 F 0 "LED5" H 9150 1600 60  0000 C CNN
 F 1 "RGB" H 9600 1600 60  0000 C CNN
-F 2 "spinny:LED_CLV1L-PLCC4" H 9400 1400 60  0001 C CNN
+F 2 "spin:LED_CLV1L-PLCC4" H 9400 1400 60  0001 C CNN
 F 3 "" H 9400 1400 60  0000 C CNN
 	1    9400 1600
@@
 F 0 "LED6" H 9150 1850 60  0000 C CNN
 F 1 "RGB" H 9600 1850 60  0000 C CNN
-F 2 "spinny:LED_CLV1L-PLCC4" H 9400 1650 60  0001 C CNN
+F 2 "spin:LED_CLV1L-PLCC4" H 9400 1650 60  0001 C CNN
 F 3 "" H 9400 1650 60  0000 C CNN
 	1    9400 1850
@@
 F 0 "LED7" H 9150 2100 60  0000 C CNN
 F 1 "RGB" H 9600 2100 60  0000 C CNN
-F 2 "spinny:LED_CLV1L-PLCC4" H 9400 1900 60  0001 C CNN
+F 2 "spin:LED_CLV1L-PLCC4" H 9400 1900 60  0001 C CNN
 F 3 "" H 9400 1900 60  0000 C CNN
 	1    9400 2100
@@
 F 0 "LED8" H 9150 2350 60  0000 C CNN
 F 1 "RGB" H 9600 2350 60  0000 C CNN
-F 2 "spinny:LED_CLV1L-PLCC4" H 9400 2150 60  0001 C CNN
+F 2 "spin:LED_CLV1L-PLCC4" H 9400 2150 60  0001 C CNN
 F 3 "" H 9400 2150 60  0000 C CNN
 	1    9400 2350
@@
 F 0 "LED9" H 9150 2600 60  0000 C CNN
 F 1 "RGB" H 9600 2600 60  0000 C CNN
-F 2 "spinny:LED_CLV1L-PLCC4" H 9400 2400 60  0001 C CNN
+F 2 "spin:LED_CLV1L-PLCC4" H 9400 2400 60  0001 C CNN
 F 3 "" H 9400 2400 60  0000 C CNN
 	1    9400 2600
@@
 F 0 "LED10" H 9150 2850 60  0000 C CNN
 F 1 "RGB" H 9600 2850 60  0000 C CNN
-F 2 "spinny:LED_CLV1L-PLCC4" H 9400 2650 60  0001 C CNN
+F 2 "spin:LED_CLV1L-PLCC4" H 9400 2650 60  0001 C CNN
 F 3 "" H 9400 2650 60  0000 C CNN
 	1    9400 2850
@@
 F 0 "LED11" H 9150 3100 60  0000 C CNN
 F 1 "RGB" H 9600 3100 60  0000 C CNN
-F 2 "spinny:LED_CLV1L-PLCC4" H 9400 2900 60  0001 C CNN
+F 2 "spin:LED_CLV1L-PLCC4" H 9400 2900 60  0001 C CNN
 F 3 "" H 9400 2900 60  0000 C CNN
 	1    9400 3100
@@
 F 0 "LED12" H 9150 3350 60  0000 C CNN
 F 1 "RGB" H 9600 3350 60  0000 C CNN
-F 2 "spinny:LED_CLV1L-PLCC4" H 9400 3150 60  0001 C CNN
+F 2 "spin:LED_CLV1L-PLCC4" H 9400 3150 60  0001 C CNN
 F 3 "" H 9400 3150 60  0000 C CNN
 	1    9400 3350
@@
 F 0 "LED13" H 9150 3600 60  0000 C CNN
 F 1 "RGB" H 9600 3600 60  0000 C CNN
-F 2 "spinny:LED_CLV1L-PLCC4" H 9400 3400 60  0001 C CNN
+F 2 "spin:LED_CLV1L-PLCC4" H 9400 3400 60  0001 C CNN
 F 3 "" H 9400 3400 60  0000 C CNN
 	1    9400 3600
@@
 F 0 "LED14" H 9150 3850 60  0000 C CNN
 F 1 "RGB" H 9600 3850 60  0000 C CNN
-F 2 "spinny:LED_CLV1L-PLCC4" H 9400 3650 60  0001 C CNN
+F 2 "spin:LED_CLV1L-PLCC4" H 9400 3650 60  0001 C CNN
 F 3 "" H 9400 3650 60  0000 C CNN
 	1    9400 3850
@@
 F 0 "LED15" H 9150 4100 60  0000 C CNN
 F 1 "RGB" H 9600 4100 60  0000 C CNN
-F 2 "spinny:LED_CLV1L-PLCC4" H 9400 3900 60  0001 C CNN
+F 2 "spin:LED_CLV1L-PLCC4" H 9400 3900 60  0001 C CNN
 F 3 "" H 9400 3900 60  0000 C CNN
 	1    9400 4100
@@
 F 0 "LED16" H 9150 4350 60  0000 C CNN
 F 1 "RGB" H 9600 4350 60  0000 C CNN
-F 2 "spinny:LED_CLV1L-PLCC4" H 9400 4150 60  0001 C CNN
+F 2 "spin:LED_CLV1L-PLCC4" H 9400 4150 60  0001 C CNN
 F 3 "" H 9400 4150 60  0000 C CNN
 	1    9400 4350
@@
 F 0 "LED17" H 10350 600 60  0000 C CNN
 F 1 "RGB" H 10800 600 60  0000 C CNN
-F 2 "spinny:LED_CLV1L-PLCC4" H 10600 400 60  0001 C CNN
+F 2 "spin:LED_CLV1L-PLCC4" H 10600 400 60  0001 C CNN
 F 3 "" H 10600 400 60  0000 C CNN
 	1    10600 600
@@
 F 0 "LED18" H 10350 850 60  0000 C CNN
 F 1 "RGB" H 10800 850 60  0000 C CNN
-F 2 "spinny:LED_CLV1L-PLCC4" H 10600 650 60  0001 C CNN
+F 2 "spin:LED_CLV1L-PLCC4" H 10600 650 60  0001 C CNN
 F 3 "" H 10600 650 60  0000 C CNN
 	1    10600 850
@@
 F 0 "LED19" H 10350 1100 60  0000 C CNN
 F 1 "RGB" H 10800 1100 60  0000 C CNN
-F 2 "spinny:LED_CLV1L-PLCC4" H 10600 900 60  0001 C CNN
+F 2 "spin:LED_CLV1L-PLCC4" H 10600 900 60  0001 C CNN
 F 3 "" H 10600 900 60  0000 C CNN
 	1    10600 1100
@@
 F 0 "LED20" H 10350 1350 60  0000 C CNN
 F 1 "RGB" H 10800 1350 60  0000 C CNN
-F 2 "spinny:LED_CLV1L-PLCC4" H 10600 1150 60  0001 C CNN
+F 2 "spin:LED_CLV1L-PLCC4" H 10600 1150 60  0001 C CNN
 F 3 "" H 10600 1150 60  0000 C CNN
 	1    10600 1350
@@
 F 0 "LED21" H 10350 1600 60  0000 C CNN
 F 1 "RGB" H 10800 1600 60  0000 C CNN
-F 2 "spinny:LED_CLV1L-PLCC4" H 10600 1400 60  0001 C CNN
+F 2 "spin:LED_CLV1L-PLCC4" H 10600 1400 60  0001 C CNN
 F 3 "" H 10600 1400 60  0000 C CNN
 	1    10600 1600
@@
 F 0 "LED22" H 10350 1850 60  0000 C CNN
 F 1 "RGB" H 10800 1850 60  0000 C CNN
-F 2 "spinny:LED_CLV1L-PLCC4" H 10600 1650 60  0001 C CNN
+F 2 "spin:LED_CLV1L-PLCC4" H 10600 1650 60  0001 C CNN
 F 3 "" H 10600 1650 60  0000 C CNN
 	1    10600 1850
@@
 F 0 "LED23" H 10350 2100 60  0000 C CNN
 F 1 "RGB" H 10800 2100 60  0000 C CNN
-F 2 "spinny:LED_CLV1L-PLCC4" H 10600 1900 60  0001 C CNN
+F 2 "spin:LED_CLV1L-PLCC4" H 10600 1900 60  0001 C CNN
 F 3 "" H 10600 1900 60  0000 C CNN
 	1    10600 2100
@@
 F 0 "LED24" H 10350 2350 60  0000 C CNN
 F 1 "RGB" H 10800 2350 60  0000 C CNN
-F 2 "spinny:LED_CLV1L-PLCC4" H 10600 2150 60  0001 C CNN
+F 2 "spin:LED_CLV1L-PLCC4" H 10600 2150 60  0001 C CNN
 F 3 "" H 10600 2150 60  0000 C CNN
 	1    10600 2350
@@
 F 0 "LED25" H 10350 2600 60  0000 C CNN
 F 1 "RGB" H 10800 2600 60  0000 C CNN
-F 2 "spinny:LED_CLV1L-PLCC4" H 10600 2400 60  0001 C CNN
+F 2 "spin:LED_CLV1L-PLCC4" H 10600 2400 60  0001 C CNN
 F 3 "" H 10600 2400 60  0000 C CNN
 	1    10600 2600
@@
 F 0 "LED26" H 10350 2850 60  0000 C CNN
 F 1 "RGB" H 10800 2850 60  0000 C CNN
-F 2 "spinny:LED_CLV1L-PLCC4" H 10600 2650 60  0001 C CNN
+F 2 "spin:LED_CLV1L-PLCC4" H 10600 2650 60  0001 C CNN
 F 3 "" H 10600 2650 60  0000 C CNN
 	1    10600 2850
@@
 F 0 "LED27" H 10350 3100 60  0000 C CNN
 F 1 "RGB" H 10800 3100 60  0000 C CNN
-F 2 "spinny:LED_CLV1L-PLCC4" H 10600 2900 60  0001 C CNN
+F 2 "spin:LED_CLV1L-PLCC4" H 10600 2900 60  0001 C CNN
 F 3 "" H 10600 2900 60  0000 C CNN
 	1    10600 3100
@@
 F 0 "LED28" H 10350 3350 60  0000 C CNN
 F 1 "RGB" H 10800 3350 60  0000 C CNN
-F 2 "spinny:LED_CLV1L-PLCC4" H 10600 3150 60  0001 C CNN
+F 2 "spin:LED_CLV1L-PLCC4" H 10600 3150 60  0001 C CNN
 F 3 "" H 10600 3150 60  0000 C CNN
 	1    10600 3350
@@
 F 0 "LED29" H 10350 3600 60  0000 C CNN
 F 1 "RGB" H 10800 3600 60  0000 C CNN
-F 2 "spinny:LED_CLV1L-PLCC4" H 10600 3400 60  0001 C CNN
+F 2 "spin:LED_CLV1L-PLCC4" H 10600 3400 60  0001 C CNN
 F 3 "" H 10600 3400 60  0000 C CNN
 	1    10600 3600
@@
 F 0 "LED30" H 10350 3850 60  0000 C CNN
 F 1 "RGB" H 10800 3850 60  0000 C CNN
-F 2 "spinny:LED_CLV1L-PLCC4" H 10600 3650 60  0001 C CNN
+F 2 "spin:LED_CLV1L-PLCC4" H 10600 3650 60  0001 C CNN
 F 3 "" H 10600 3650 60  0000 C CNN
 	1    10600 3850
@@
 F 0 "LED31" H 10350 4100 60  0000 C CNN
 F 1 "RGB" H 10800 4100 60  0000 C CNN
-F 2 "spinny:LED_CLV1L-PLCC4" H 10600 3900 60  0001 C CNN
+F 2 "spin:LED_CLV1L-PLCC4" H 10600 3900 60  0001 C CNN
 F 3 "" H 10600 3900 60  0000 C CNN
 	1    10600 4100
@@
 F 0 "LED32" H 10350 4350 60  0000 C CNN
 F 1 "RGB" H 10800 4350 60  0000 C CNN
-F 2 "spinny:LED_CLV1L-PLCC4" H 10600 4150 60  0001 C CNN
+F 2 "spin:LED_CLV1L-PLCC4" H 10600 4150 60  0001 C CNN
 F 3 "" H 10600 4150 60  0000 C CNN
 	1    10600 4350

Commit message: Working on pcb
Parts:
- C1, C2, C3, C4: footprint Capacitors_SMD:C_0805_HandSoldering -> Capacitors_SMD:C_0603_HandSoldering
- C10, C6, C7, C8, C9: footprint (none) -> Capacitors_SMD:C_0603_HandSoldering
- L1: footprint (none) -> spin:SRU1028-10x10-Octogon
- P2, P3, P4, P5: footprint (none) -> Socket_Strips:Socket_Strip_Straight_1x01
- R1, R2, R3, R4, R5: footprint Resistors_SMD:R_0805_HandSoldering -> Resistors_SMD:R_0603_HandSoldering
- R6, R7: footprint (none) -> Resistors_SMD:R_0603_HandSoldering
- SW5: footprint (none) -> Buttons_Switches_SMD:SW_SPST_EVQPE1
- U1: value STM32F410R8-LQFP64 -> STM32F410R8/B
- U5: footprint (none) -> TO_SOT_Packages_SMD:SOT-223
- U6: footprint (none) -> spin:WSON-8_2x2mm
Connections:
- net labels removed: ADC1, ADC2, ADC3
- no-connect marks 36 -> 39
Changed lines of the file:
@@
 LIBS:contrib
 LIBS:valves
+LIBS:prototype1-cache
 EELAYER 25 0
 EELAYER END
@@
 F 0 "C1" H 1825 1200 50  0000 L CNN
 F 1 "100n" H 1825 1000 50  0000 L CNN
-F 2 "Capacitors_SMD:C_0805_HandSoldering" H 1838 950 50  0001 C CNN
+F 2 "Capacitors_SMD:C_0603_HandSoldering" H 1838 950 50  0001 C CNN
 F 3 "" H 1800 1100 50  0000 C CNN
 	1    1800 1100
@@
 F 0 "C2" H 2125 1200 50  0000 L CNN
 F 1 "100n" H 2125 1000 50  0000 L CNN
-F 2 "Capacitors_SMD:C_0805_HandSoldering" H 2138 950 50  0001 C CNN
+F 2 "Capacitors_SMD:C_0603_HandSoldering" H 2138 950 50  0001 C CNN
 F 3 "" H 2100 1100 50  0000 C CNN
 	1    2100 1100
@@
 F 0 "C3" H 2425 1200 50  0000 L CNN
 F 1 "100n" H 2425 1000 50  0000 L CNN
-F 2 "Capacitors_SMD:C_0805_HandSoldering" H 2438 950 50  0001 C CNN
+F 2 "Capacitors_SMD:C_0603_HandSoldering" H 2438 950 50  0001 C CNN
 F 3 "" H 2400 1100 50  0000 C CNN
 	1    2400 1100
@@
 F 0 "C4" H 2725 1200 50  0000 L CNN
 F 1 "100n" H 2725 1000 50  0000 L CNN
-F 2 "Capacitors_SMD:C_0805_HandSoldering" H 2738 950 50  0001 C CNN
+F 2 "Capacitors_SMD:C_0603_HandSoldering" H 2738 950 50  0001 C CNN
 F 3 "" H 2700 1100 50  0000 C CNN
 	1    2700 1100
@@
 F 0 "R3" V 8680 800 50  0000 C CNN
 F 1 "300" V 8600 800 50  0000 C CNN
-F 2 "Resistors_SMD:R_0805_HandSoldering" V 8530 800 50  0001 C CNN
+F 2 "Resistors_SMD:R_0603_HandSoldering" V 8530 800 50  0001 C CNN
 F 3 "" H 8600 800 50  0000 C CNN
 	1    8600 800
@@
 F 0 "R4" V 8680 2250 50  0000 C CNN
 F 1 "500" V 8600 2250 50  0000 C CNN
-F 2 "Resistors_SMD:R_0805_HandSoldering" V 8530 2250 50  0001 C CNN
+F 2 "Resistors_SMD:R_0603_HandSoldering" V 8530 2250 50  0001 C CNN
 F 3 "" H 8600 2250 50  0000 C CNN
 	1    8600 2250
@@
 F 0 "R5" V 8680 3700 50  0000 C CNN
 F 1 "500" V 8600 3700 50  0000 C CNN
-F 2 "Resistors_SMD:R_0805_HandSoldering" V 8530 3700 50  0001 C CNN
+F 2 "Resistors_SMD:R_0603_HandSoldering" V 8530 3700 50  0001 C CNN
 F 3 "" H 8600 3700 50  0000 C CNN
 	1    8600 3700
@@
 F 0 "R1" V 2130 3600 50  0000 C CNN
 F 1 "22" V 2050 3600 50  0000 C CNN
-F 2 "Resistors_SMD:R_0805_HandSoldering" V 1980 3600 50  0001 C CNN
+F 2 "Resistors_SMD:R_0603_HandSoldering" V 1980 3600 50  0001 C CNN
 F 3 "" H 2050 3600 50  0000 C CNN
 	1    2050 3600
@@
 F 0 "R2" V 2130 3800 50  0000 C CNN
 F 1 "22" V 2050 3800 50  0000 C CNN
-F 2 "Resistors_SMD:R_0805_HandSoldering" V 1980 3800 50  0001 C CNN
+F 2 "Resistors_SMD:R_0603_HandSoldering" V 1980 3800 50  0001 C CNN
 F 3 "" H 2050 3800 50  0000 C CNN
 	1    2050 3800
@@
 U 1 1 575503AA
 P 1050 3900
-F 0 "U1" H 1050 7250 60  0000 C CNN
-F 1 "STM32F410R8-LQFP64" H 1050 500 60  0000 C CNN
+F 0 "U1" H 850 3900 60  0000 C CNN
+F 1 "STM32F410R8/B" H 1000 550 60  0000 C CNN
 F 2 "Housings_QFP:TQFP-64_10x10mm_Pitch0.5mm" H 1350 6250 60  0001 C CNN
 F 3 "" H 1350 6250 60  0000 C CNN
@@
 F 0 "U5" H 3350 2950 50  0000 C CNN
 F 1 "LM1117-3.3" H 3250 3450 50  0000 C CNN
-F 2 "" H 3250 3200 50  0000 C CNN
+F 2 "TO_SOT_Packages_SMD:SOT-223" H 3250 3200 50  0001 C CNN
 F 3 "" H 3250 3200 50  0000 C CNN
 	1    3250 3200
@@
 F 0 "SW5" H 3100 7600 50  0000 C CNN
 F 1 "SPST" H 3100 7400 50  0000 C CNN
-F 2 "" H 3100 7500 50  0000 C CNN
+F 2 "Buttons_Switches_SMD:SW_SPST_EVQPE1" H 3100 7500 50  0001 C CNN
 F 3 "" H 3100 7500 50  0000 C CNN
 	1    3100 7500
@@
 F 0 "P2" H 2150 7100 50  0000 C CNN
 F 1 "AAA1 HOT" V 2250 7000 50  0000 C CNN
-F 2 "" H 2150 7000 50  0000 C CNN
+F 2 "Socket_Strips:Socket_Strip_Straight_1x01" H 2150 7000 50  0001 C CNN
 F 3 "" H 2150 7000 50  0000 C CNN
 	1    2150 7000
@@
 F 0 "P3" H 2150 7400 50  0000 C CNN
 F 1 "AAA1 GND" V 2250 7300 50  0000 C CNN
-F 2 "" H 2150 7300 50  0000 C CNN
+F 2 "Socket_Strips:Socket_Strip_Straight_1x01" H 2150 7300 50  0001 C CNN
 F 3 "" H 2150 7300 50  0000 C CNN
 	1    2150 7300
@@
 F 0 "P4" H 2600 7100 50  0000 C CNN
 F 1 "AAA2 GND" V 2700 7000 50  0000 C CNN
-F 2 "" H 2600 7000 50  0000 C CNN
+F 2 "Socket_Strips:Socket_Strip_Straight_1x01" H 2600 7000 50  0001 C CNN
 F 3 "" H 2600 7000 50  0000 C CNN
 	1    2600 7000
@@
 F 0 "P5" H 2600 7400 50  0000 C CNN
 F 1 "AAA2 HOT" V 2700 7300 50  0000 C CNN
-F 2 "" H 2600 7300 50  0000 C CNN
+F 2 "Socket_Strips:Socket_Strip_Straight_1x01" H 2600 7300 50  0001 C CNN
 F 3 "" H 2600 7300 50  0000 C CNN
 	1    2600 7300
@@
 Text Notes 2600 4700 0    60   ~ 0
 Resistors here???
-Text GLabel 1550 2650 2    60   Input ~ 0
-ADC1
-Text GLabel 1550 2750 2    60   Input ~ 0
-ADC2
-Text GLabel 1550 2850 2    60   Input ~ 0
-ADC3
 $Comp
 L TPS61021 U6
@@
 F 0 "U6" H 4300 8950 60  0000 C CNN
 F 1 "TPS61021" H 4200 8450 60  0000 C CNN
-F 2 "" H 5000 7750 60  0000 C CNN
+F 2 "spin:WSON-8_2x2mm" H 5000 7750 60  0001 C CNN
 F 3 "" H 5000 7750 60  0000 C CNN
 	1    5000 7750
@@
 F 0 "L1" V 4850 6800 50  0000 C CNN
 F 1 "1uH 4.9mOhm" V 5050 6800 50  0000 C CNN
-F 2 "" H 4950 6800 50  0000 C CNN
+F 2 "spin:SRU1028-10x10-Octogon" H 4950 6800 50  0001 C CNN
 F 3 "" H 4950 6800 50  0000 C CNN
 	1    4950 6800
@@
 F 0 "C10" H 5275 6600 50  0000 L CNN
 F 1 "10u" H 5275 6400 50  0000 L CNN
-F 2 "" H 5288 6350 50  0000 C CNN
+F 2 "Capacitors_SMD:C_0603_HandSoldering" H 5288 6350 50  0001 C CNN
 F 3 "" H 5250 6500 50  0000 C CNN
 	1    5250 6500
@@
 F 0 "C9" H 3575 7150 50  0000 L CNN
 F 1 "10u" H 3575 6950 50  0000 L CNN
-F 2 "" H 3588 6900 50  0000 C CNN
+F 2 "Capacitors_SMD:C_0603_HandSoldering" H 3588 6900 50  0001 C CNN
 F 3 "" H 3550 7050 50  0000 C CNN
 	1    3550 7050
@@
 F 0 "C8" H 3375 7150 50  0000 L CNN
 F 1 "10u" H 3375 6950 50  0000 L CNN
-F 2 "" H 3388 6900 50  0000 C CNN
+F 2 "Capacitors_SMD:C_0603_HandSoldering" H 3388 6900 50  0001 C CNN
 F 3 "" H 3350 7050 50  0000 C CNN
 	1    3350 7050
@@
 F 0 "R7" V 3630 6600 50  0000 C CNN
 F 1 "100k" V 3550 6600 50  0000 C CNN
-F 2 "" V 3480 6600 50  0000 C CNN
+F 2 "Resistors_SMD:R_0603_HandSoldering" V 3480 6600 50  0001 C CNN
 F 3 "" H 3550 6600 50  0000 C CNN
 	1    3550 6600
@@
 F 0 "R6" V 3380 6750 50  0000 C CNN
 F 1 "316k" V 3300 6750 50  0000 C CNN
-F 2 "" V 3230 6750 50  0000 C CNN
+F 2 "Resistors_SMD:R_0603_HandSoldering" V 3230 6750 50  0001 C CNN
 F 3 "" H 3300 6750 50  0000 C CNN
 	1    3300 6750
@@
 F 0 "C6" H 3125 6850 50  0000 L CNN
 F 1 "24p" H 3125 6650 50  0000 L CNN
-F 2 "" H 3138 6600 50  0000 C CNN
+F 2 "Capacitors_SMD:C_0603_HandSoldering" H 3138 6600 50  0001 C CNN
 F 3 "" H 3100 6750 50  0000 C CNN
 	1    3100 6750
@@
 F 0 "C7" H 3175 7150 50  0000 L CNN
 F 1 "10u" H 3175 6950 50  0000 L CNN
-F 2 "" H 3188 6900 50  0000 C CNN
+F 2 "Capacitors_SMD:C_0603_HandSoldering" H 3188 6900 50  0001 C CNN
 F 3 "" H 3150 7050 50  0000 C CNN
 	1    3150 7050
@@
 Wire Wire Line
 	3700 6400 3700 6650
+NoConn ~ 1550 2650
+NoConn ~ 1550 2750
+NoConn ~ 1550 2850
+$Comp
+L GND #PWR?
+U 1 1 575D2EAF
+P 3950 6400
+F 0 "#PWR?" H 3950 6150 50  0001 C CNN
+F 1 "GND" H 3950 6250 50  0000 C CNN
+F 2 "" H 3950 6400 50  0000 C CNN
+F 3 "" H 3950 6400 50  0000 C CNN
+	1    3950 6400
+	1    0    0    -1
+$EndComp
+Connection ~ 3950 6400
 $EndSCHEMATC

Commit message: More pcb changes
Other:
- note added: "ADD:\nFlash"
Changed lines of the file:
@@
 Text Notes 6950 5050 0    60   ~ 0
 NOTE: VIAs to ground under TLC5926.\nFor heat. See datasheet.
-Text Notes 6050 6050 0    60   ~ 0
+Text Notes 6050 6750 0    60   ~ 0
 ADD:\nAccelerometers
 Text Notes 6050 7000 0    60   ~ 0
@@
 $EndComp
 Connection ~ 3950 6400
+Text Notes 6050 6500 0    60   ~ 0
+ADD:\nFlash
 $EndSCHEMATC

Commit message: More pcb changes
Parts:
- removed U1: STM32F410R8/B, Housings_QFP:TQFP-64_10x10mm_Pitch0.5mm, symbol STM32F410R8-LQFP64
- removed U5: LM1117-3.3, TO_SOT_Packages_SMD:SOT-223, symbol LM1117-3.3
- added C11: 100n, Capacitors_SMD:C_0603_HandSoldering, symbol C
- added C12: 10u, Capacitors_SMD:C_0603_HandSoldering, symbol C
- added U1: STM32F410R8/B, Housings_QFP:TQFP-64_10x10mm_Pitch0.5mm, symbol STM32F410R8/B
- added U5: LD1117S33CTR, TO_SOT_Packages_SMD:SOT-223, symbol LD1117S33CTR
- added U7: L3GD20HTR, spin:L3GD20H, symbol L3GD20HTR
- added U8, U9: LIS331HH, spin:LGA16, symbol LIS331HH
- C1, C2, C3, C4: manf# (none) -> 885012206071
- C5: manf# (none) -> VJ0805G475KXYTW1BC
- L1: manf# (none) -> SRU1028-1R0Y
- LED1, LED10, LED11, LED12, LED13, LED14, LED15, LED16, LED17, LED18, LED19, LED2, LED20, LED21, LED22, LED23, LED24, LED25, LED26, LED27, LED28, LED29, LED3, LED30, LED31, LED32, LED4, LED5, LED6, LED7, LED8, LED9: manf# (none) -> CLV1L-FKB-CHMMQDGBB7673673
- P1: footprint Connect:USB_Micro-B -> spin:ZX62M-B-5P; manf# (none) -> ZX62M-B-5P(30)
- R1, R2: manf# (none) -> ERJ-3EKF22R0V
- R3, R4, R5: footprint Resistors_SMD:R_0603_HandSoldering -> Resistors_ThroughHole:Resistor_Vertical_RM5mm
- SW1: value UP/BOOT -> Boot Button; footprint Buttons_Switches_SMD:SW_SPST_B3U-1000P -> spin:Button; manf# (none) -> 2-1437565-8
- SW2: value LEFT -> Button; footprint Buttons_Switches_SMD:SW_SPST_B3U-1000P -> spin:Button; manf# (none) -> 2-1437565-8
- SW3: value RIGHT -> Button; footprint Buttons_Switches_SMD:SW_SPST_B3U-1000P -> spin:Button; manf# (none) -> 2-1437565-8
- SW4: value DOWN -> Button; footprint Buttons_Switches_SMD:SW_SPST_B3U-1000P -> spin:Button; manf# (none) -> 2-1437565-8
- SW5: footprint Buttons_Switches_SMD:SW_SPST_EVQPE1 -> (none); manf# (none) -> OS102011MA1QN1C
- U2, U3, U4: manf# (none) -> TLC5926IPWPR
- U6: manf# (none) -> TPS61021DSGT
Connections:
- net labels added: SS_ACC1, SS_ACC2, SS_GYRO
- wire segments 51 -> 69
- no-connect marks 39 -> 35
Other:
- note removed: "ADD:\nAccelerometers"

Commit message: pcb schematic almost done!
Parts:
- removed C7, C9: 10u, Capacitors_SMD:C_0603_HandSoldering, symbol C
- added 1k1, 1k2, 1k3, 1k4: R, Resistors_SMD:R_0805_HandSoldering, symbol R
- added C11, C14, C18, C19, C20, C6: 10u, Capacitors_SMD:C_0805_HandSoldering, symbol C
- added C13, C15, C16, C21: 100n, Capacitors_SMD:C_0603_HandSoldering, symbol C
- added C17: 10n, Capacitors_SMD:C_0805_HandSoldering, symbol C
- added D?: LED, LEDs:LED_0603, symbol LED
- added R?: 100, Resistors_SMD:R_0805_HandSoldering, symbol R
- added U10: AT25_EEPROM, Housings_SOIC:SOIC-8_3.9x4.9mm_Pitch1.27mm, symbol AT25_EEPROM
- C10, C12: footprint Capacitors_SMD:C_0603_HandSoldering -> Capacitors_SMD:C_0805_HandSoldering; manf# (none) -> LMK212BJ106KD-T
- C8: value 10u -> 4.7u; footprint Capacitors_SMD:C_0603_HandSoldering -> Capacitors_SMD:C_0805_HandSoldering; manf# (none) -> VJ0805G475KXYTW1BC
- C9: renamed from C6; value 24p -> 22p; footprint Capacitors_SMD:C_0603_HandSoldering -> Capacitors_SMD:C_0805_HandSoldering; manf# (none) -> C0805C220K3GACTU
- P1: renamed from P2; footprint Socket_Strips:Socket_Strip_Straight_1x01 -> (none)
- P2: renamed from P3; footprint Socket_Strips:Socket_Strip_Straight_1x01 -> (none)
- P3: renamed from P4; footprint Socket_Strips:Socket_Strip_Straight_1x01 -> (none)
- P4: renamed from P5; footprint Socket_Strips:Socket_Strip_Straight_1x01 -> (none)
- R3: renamed from R6; footprint Resistors_SMD:R_0603_HandSoldering -> Resistors_SMD:R_1206_HandSoldering; manf# (none) -> ERJ-8ENF3163V
- R4: renamed from R7; footprint Resistors_SMD:R_0603_HandSoldering -> Resistors_SMD:R_0805_HandSoldering; manf# (none) -> CRCW0805100KFKEA
- SW2: renamed from SW1; value Boot Button -> Button
- U1: footprint Housings_QFP:TQFP-64_10x10mm_Pitch0.5mm -> spin:STM32F410-LQFP64
- U7: renamed from U2; footprint Housings_SSOP:SSOP-24_3.9x8.7mm_Pitch0.635mm -> spin:TLC5926
- U8: renamed from U3; footprint Housings_SSOP:SSOP-24_3.9x8.7mm_Pitch0.635mm -> spin:TLC5926
- U9: renamed from U4; footprint Housings_SSOP:SSOP-24_3.9x8.7mm_Pitch0.635mm -> spin:TLC5926
- renumbered C11 to C3, C3 to C4, C4 to C5, C5 to C7, P1 to P5, R3 to R5, R4 to R6, R5 to R7, SW5 to SW1, SW2 to SW3, SW3 to SW4, SW4 to SW5, U5 to U2, U6 to U3, U7 to U4, U8 to U5, U9 to U6
Connections:
- net BOOT0: now also 1k1.2; no longer SW2.1
- net GND: now also C10.2, C8.1, U4.8 (DEN), C11.2, C13.2, C14.2, C15.2, C16.2, C17.2, C18.2, C19.2, C20.1, C21.2, C6.2, D?.1 (K), U10.4 (GND); no longer C10.1, C8.2, U4.15 (Vdd)
- net MISO1: now also U10.2 (MISO)
- net MOSI1: now also U10.5 (MOSI)
- net SCK1: now also U10.6 (SCK)
- net at L1.2, SW1.2, U3.5 (VIN)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: now also C20.2; no longer C10.2
- net +3V3: now reaches U1.1 (VBAT)
- net +3V3: now also C1.1, C10.1, C12.1, C2.1, C4.1, C5.1, C7.1, C9.2, LED1.1 (A), LED10.1 (A), LED11.1 (A), LED12.1 (A), LED13.1 (A), LED14.1 (A), LED15.1 (A), LED16.1 (A), LED17.1 (A), LED18.1 (A), LED19.1 (A), LED2.1 (A), LED20.1 (A), LED21.1 (A), LED22.1 (A), LED23.1 (A), LED24.1 (A), LED25.1 (A), LED26.1 (A), LED27.1 (A), LED28.1 (A), LED29.1 (A), LED3.1 (A), LED30.1 (A), LED31.1 (A), LED32.1 (A), LED4.1 (A), LED5.1 (A), LED6.1 (A), LED7.1 (A), LED8.1 (A), LED9.1 (A), R3.2, SW2.2, SW3.2, SW4.2, SW5.2, U1.13 (VDDA/VREF+), U1.19 (VDD), U1.32 (VDD), U1.48 (VDD), U1.64 (VDD), U1.7 (NRST), U2.2 (VO), U3.3 (VOUT), U3.4 (VOUT), U4.1 (Vdd_IO), U4.15 (Vdd), U4.16 (Vdd), U5.1 (Vdd_IO), U5.14 (Vdd), U5.15 (Vdd), U6.1 (Vdd_IO), U6.14 (Vdd), U6.15 (Vdd), U7.24 (VDD), U8.24 (VDD), U9.24 (VDD), C11.1, C13.1, C14.1, C15.1, C16.1, C18.1, C19.1, C21.1, C6.1, U10.8 (Vcc)
- net at SW3.1: now also 1k2.1; no longer U1.27 (PB1)
- net at SW4.1: now also 1k3.1; no longer U1.28 (PB2)
- net SS_FLASH: now reaches U1.38 (PC7)
- net SS_FLASH: now also U10.1 (~CS)
- net FLASH_WP: now reaches U1.39 (PC8)
- net FLASH_WP: now also U10.3 (~WP)
- net FLASH_HOLD: now reaches U1.40 (PC9)
- net FLASH_HOLD: now also U10.7 (~HOLD)
- net at SW5.1: now also 1k4.1; no longer U1.55 (PB3)
- net LED1: now reaches U1.56 (PB4)
- net LED1: now also R?.2
- net at U4.14 (Cap): now also C17.1
- removed net VCC: C1.1, C12.1, C2.1, C4.1, C5.1, C7.1, C8.1, C9.2, LED1.1 (A), LED10.1 (A), LED11.1 (A), LED12.1 (A), LED13.1 (A), LED14.1 (A), LED15.1 (A), LED16.1 (A), LED17.1 (A), LED18.1 (A), LED19.1 (A), LED2.1 (A), LED20.1 (A), LED21.1 (A), LED22.1 (A), LED23.1 (A), LED24.1 (A), LED25.1 (A), LED26.1 (A), LED27.1 (A), LED28.1 (A), LED29.1 (A), LED3.1 (A), LED30.1 (A), LED31.1 (A), LED32.1 (A), LED4.1 (A), LED5.1 (A), LED6.1 (A), LED7.1 (A), LED8.1 (A), LED9.1 (A), R3.2, SW2.2, SW3.2, SW4.2, SW5.2, U1.13 (VDDA/VREF+), U1.19 (VDD), U1.30 (VCAP_1), U1.32 (VDD), U1.48 (VDD), U1.64 (VDD), U2.2 (VO), U3.3 (VOUT), U3.4 (VOUT), U4.1 (Vdd_IO), U4.16 (Vdd), U5.1 (Vdd_IO), U5.14 (Vdd), U5.15 (Vdd), U6.1 (Vdd_IO), U6.14 (Vdd), U6.15 (Vdd), U7.24 (VDD), U8.24 (VDD), U9.24 (VDD)
- new net: 1k1.1, SW2.1
- new net: C8.2, U1.30 (VCAP_1)
- new net: D?.2 (A), R?.1
- new net BUT2: 1k2.2, U1.27 (PB1)
- new net BUT3: 1k3.2, U1.28 (PB2)
- new net BUT4: 1k4.2, U1.55 (PB3)
Other:
- note added: "100n cap near each Vdd!"
- note added: "10n cap "must guarantee 1nF value under 12V bias condition""
- note added: "4.7u cap near V_CAP1!"
- note added: "ADD:\nCrystal(s)?"
- note added: "Datasheet says aluminum caps for the 10uF ones.\nDon't know why; using ceramic for now."
- note added: "Place caps near Vdd!"
- note added: "Place caps near pin 14!"
- note added: "See datasheet for circuit placement!"
- note removed: "???"
- note removed: "????"
- note removed: "ADD:\nFlash"
- note removed: "NOTE: VIAs to ground under TLC5926.\nFor heat. See datasheet."
- note removed: "Rearrange caps?"
- note removed: "Resistors here???"
- note removed: "Use these pins or others?"
- moved on the sheet: C3, SW2, SW3, SW4, SW5, U2, U4, U5, U6
