File: pcb/prototype1/prototype1.kicad_pcb (KiCad board)
At the start: 2 copper layers, 73.4 x 73.4 mm, 87 parts, among them P5 USB_B, SW2 Button, SW3 Button, SW4 Button, SW5 Button, U1 STM32F401, U10 AT25_EEPROM, U11 LD1117S33CTR, U2 MP34DT01-M, U3 L3GD20HTR, U4 LIS331HH, U5 LIS331HH, U6 TPS61021, U7 TLC5926, U8 TLC5926, U9 TLC5926

Commit message: Working on schematic
Parts:
- LED17, LED18, LED19, LED20, LED21, LED22, LED23, LED24, LED25, LED26, LED27, LED28, LED29, LED30, LED31, LED32, U8: moved to B.Cu
- U9: moved to F.Cu
- moved LED12 157.8 mm to (150.0, 66.0)
- moved LED10 153.0 mm to (150.0, 72.0)
- moved LED15 151.2 mm to (150.0, 57.0)
- moved LED30 146.9 mm to (150.0, 60.0)
- moved LED24 146.6 mm to (150.0, 78.0)
- moved LED8 141.6 mm to (150.0, 78.0)
- moved LED31 138.7 mm to (150.0, 57.0)
- moved LED27 136.6 mm to (150.0, 69.0)
- moved LED1 134.5 mm to (150.0, 99.0)
- moved LED22 134.4 mm to (150.0, 84.0)
- moved LED16 130.6 mm to (150.0, 54.0)
- moved U2 130.4 mm to (150.0, 102.8)
- moved LED13 129.6 mm to (150.0, 63.0)
- moved LED20 126.4 mm to (150.0, 90.0)
- moved LED32 125.4 mm to (150.0, 54.0)
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Other:
- board size 73.4 x 73.4 mm -> 95.1 x 95 mm

Commit message: Working on pcb
Parts:
- C1, C10, C11, C12, C15, C18, C19, C2, C20, C21, C22, C23, C24, C25, C3, C4, C5, C6, C7, C8, C9, L1, R1, R2, R9, U1, U10, U11, U3, U6: moved to B.Cu
- moved C11 166.5 mm to (160.1, 103.8), turned to 270 degrees
- moved C22 164.1 mm to (157.9, 100.6), turned to 180 degrees
- moved C12 163.5 mm to (162.0, 104.2), turned to 270 degrees
- moved C23 157.8 mm to (137.8, 80.0)
- moved C21 155.1 mm to (141.4, 99.8)
- moved C15 152.7 mm to (164.1, 104.2), turned to 270 degrees
- moved C2 151.8 mm to (152.7, 107.1), turned to 270 degrees
- moved L1 147.4 mm to (139.0, 86.5), turned to 90 degrees
- moved C1 142.6 mm to (140.6, 113.1), turned to 180 degrees
- moved C4 138.4 mm to (147.4, 107.3), turned to 90 degrees
- moved U3 137.3 mm to (162.0, 100.0)
- moved C5 136.9 mm to (147.7, 102.6), turned to 180 degrees
- moved U11 134.6 mm to (150.0, 134.0), turned to 180 degrees
- moved C6 134.6 mm to (154.4, 107.1), turned to 90 degrees
- moved U1 133.2 mm to (150.0, 116.0)
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Other:
- outline, holes or cut-outs redrawn

Commit message: Workin on pcb!
Parts:
- added P1: AAA1 HOT, spin:test_pin, F.Cu at (177.0, 132.0)
- added P2: AAA1 GND, spin:test_pin, F.Cu at (177.0, 68.0)
- added P3: AAA2 GND, spin:test_pin, F.Cu at (123.0, 132.0)
- added P4: AAA2 HOT, spin:test_pin, F.Cu at (123.0, 68.0)
- added SW1: SPST, Buttons_Switches_ThroughHole:SW_DIP_x1_Slide, F.Cu at (143.5, 55.6)
- moved C14 153.7 mm to (158.7, 101.9)
- moved C13 145.7 mm to (141.3, 98.1), turned to 180 degrees
- moved C17 142.3 mm to (159.1, 100.0)
- moved C16 132.6 mm to (140.9, 100.0), turned to 180 degrees
- moved U5 122.7 mm to (155.0, 100.0), turned to 270 degrees
- moved U4 117.3 mm to (145.0, 100.0), turned to 90 degrees
- moved C22 0.64 mm to (158.4, 101.0)

Commit message: pcb stuff
Parts:
- added H1: Hole, spin:Hole-3mm, F.Cu at (146.0, 100.0)
- added H2: Hole, spin:Hole-3mm, F.Cu at (154.0, 100.0)
- added H3: Hole, spin:Hole-3mm, F.Cu at (114.0, 76.0)
- added H4: Hole, spin:Hole-3mm, F.Cu at (114.0, 124.0)
- added H5: Hole, spin:Hole-3mm, F.Cu at (186.0, 76.0)
- added H6: Hole, spin:Hole-3mm, F.Cu at (186.0, 124.0)
- C5, C7: moved to F.Cu
- SW1: footprint Buttons_Switches_ThroughHole:SW_DIP_x1_Slide -> spin:EVP-AYG0BA
- moved SW1 13.2 mm to (131.2, 60.3), turned to 27 degrees
- moved D1 5.24 mm to (159.5, 142.6), turned to 90 degrees
- moved U4 5.00 mm to (140.0, 100.0)
- moved U5 5.00 mm to (160.0, 100.0)
- moved C16 4.90 mm to (136.0, 100.1)
- moved C17 4.90 mm to (164.0, 100.1)
- moved C13 4.80 mm to (136.5, 98.2)
- moved C14 4.80 mm to (163.5, 102.0)
- moved R7 3.75 mm to (162.2, 139.1)
- moved U7 2.20 mm to (143.2, 76.5)
- moved U8 2.20 mm to (156.8, 76.5)
- moved U9 2.20 mm to (156.8, 76.5)
- moved C23 1.99 mm to (139.0, 78.5), turned to 270 degrees
- moved C7 1.65 mm to (146.5, 104.5)
- moved C5 1.65 mm to (146.1, 102.7)
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Connections:
- P4 pad 1: Net-(P4-Pad1) -> Net-(C23-Pad2)
- SW1 pad 1: Net-(P4-Pad1) -> Net-(C23-Pad2)
- SW1 pad 2: Net-(C23-Pad2) -> Net-(SW1-Pad2)
- U6 pad 8: Net-(C23-Pad2) -> Net-(SW1-Pad2)
Routing:
- net Net-(P1-Pad1): track 0.00 -> 49.2 mm, vias 0 -> 2
- net Net-(C23-Pad2): track 0.00 -> 45.9 mm
- net GND: track 0.00 -> 40.4 mm, vias 0 -> 2
- net Net-(SW1-Pad2): track 0.00 -> 35.6 mm, vias 0 -> 1
- net B16: track 0.00 -> 26.5 mm, vias 0 -> 1
- net B1: track 0.00 -> 26.4 mm, vias 0 -> 1
- net +3V3: track 0.00 -> 25.0 mm, vias 0 -> 5
- net G16: track 0.00 -> 24.7 mm, vias 0 -> 1
- net R1: track 0.00 -> 24.5 mm, vias 0 -> 1
- net R16: track 0.00 -> 24.4 mm, vias 0 -> 1
- net G1: track 0.00 -> 24.4 mm, vias 0 -> 1
- net B15: track 0.00 -> 23.2 mm, vias 0 -> 1
- net R2: track 0.00 -> 21.8 mm, vias 0 -> 1
- net G2: track 0.00 -> 21.6 mm, vias 0 -> 1
- net G15: track 0.00 -> 21.4 mm, vias 0 -> 1
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- added copper zone on F.Cu, net +3V3
- added copper zone on B.Cu, net GND
Other:
- net class Big added: clearance 0.4, trace_width 0.5, via_dia 0.8, via_drill 0.6
